File: final_work/全方向ワイヤレス給電.kicad_sch (KiCad schematic)
At the start: 0 parts

Commit message: 中間レポート完成
Parts:
- added C1: 0.22u, Passive_Robotech:1005, symbol Passive_Robotech:C
- added C2, C3: 0.01u, Passive_Robotech:1005, symbol Passive_Robotech:C
- added C4, C8: 0.3u, Passive_Robotech:1005, symbol Passive_Robotech:C
- added C5: 0.33u, Passive_Robotech:1005, symbol Passive_Robotech:C
- added C6: 2.2u, Passive_Robotech:1005, symbol Passive_Robotech:C
- added C7: ~, Passive_Robotech:TP-TYPEV-K16, symbol Passive_Robotech:CC
- added D1, D4: D_Zener, symbol Device:D_Zener
- added D10, D12: ~, Diode_Robotech:LED3, symbol Diode_Robotech:LED
- added D11, D2, D3, D5, D6, D7, D8: D_Schottky, symbol Device:D_Schottky
- added D9: D_Zener 12V, symbol Device:D_Zener
- added IC1: NJM2845DL1-, IC_Robotech:TO-252-3, symbol IC_Robotech:NJM2845DL1-*
- added L1, L3: 68u, Passive_Robotech:0204_slash_5, symbol Passive_Robotech:L
- added L2, L4, L5: 6.2u, Passive_Robotech:0204_slash_5, symbol Passive_Robotech:L
- added Q1, Q2: NMOS, symbol Simulation_SPICE:NMOS
- added R1, R2, R3: 100, Passive_Robotech:0204_slash_5, symbol Passive_Robotech:R
- added R4, R5: 1k, Passive_Robotech:0204_slash_5, symbol Passive_Robotech:R
- added TP1, TP2, TP3, TP4: TestPoint, symbol Connector:TestPoint
- added V_OUT: ~, Connector_Robotech:5251-02-A, symbol Connector_Robotech:MOLEX-5251-02
Connections:
- new net: D12.A, R5.2
- new net: C8.2, D12.K, L5.1
- new net: C7.+, D5.1 (K), D6.1 (K), R3.1
- new net: C4.1, D5.2 (A), D7.1 (K), L4.2
- new net: C5.2, C6.2, C7.-, D10.K, D7.2 (A), D8.2 (A), D9.2 (A), IC1.2 (GND), V_OUT.2 (S)
- new net: C6.1, IC1.3 (OUT), R4.2, V_OUT.1 (S)
- new net: C3.1, D3.2 (A), D4.1 (K), Q1.2 (G), R1.2
- new net: C2.1, D1.1 (K), D2.2 (A), Q2.2 (G), R2.2
- new net: C5.1, D9.1 (K), IC1.1 (IN), R3.2
- new net: D10.A, R4.1
- new net: D11.1 (K), R5.1
- new net: C8.1, D11.2 (A), L5.2
- new net: C4.2, D6.2 (A), D8.1 (K), L4.1
- new net +5V: L1.1, L3.1, TP3.1
- new net GND: D1.2 (A), D4.2 (A), Q1.3 (S), Q2.3 (S), TP4.1
- new net Tx+: C1.1, C2.2, D2.1 (K), L2.1, L3.2, Q1.1 (D), R2.1, TP1.1
- new net Tx-: C1.2, C3.2, D3.1 (K), L1.2, L2.2, Q2.1 (D), R1.1, TP2.1
Other:
- note added: "Receiver"
- note added: "Receiver_test"
- note added: "Transmitter"
- note removed: "Oscillator"
